File: PCB/Diesel_Injector_Tester/Diesel_Injector_Tester.kicad_pcb (KiCad board)
At the start: 2 copper layers, 35 parts, among them J1 PWR, J2 INJECTOR, J3 PROG, Q1 IRLR8726, SW1 ENABLE, SW2 PERIOD, U1 LM1117DT-3.3, U2 STM32F030F4Px, U3 MCP1416, Y1 8MHz

Commit message: PCB prepared, schematic updated
Parts:
- C10, C11, C12, C3, C4, C6, C7, C8, C9: footprint Capacitor_SMD:C_1206_3216Metric_Pad1.33x1.80mm_HandSolder -> Capacitor_SMD:C_0805_2012Metric_Pad1.18x1.45mm_HandSolder
- D2: moved to F.Cu
- D3: value GREEN -> PWR_GREEN
- D4: value GREEN -> ENABLE_GREEN
- D5: value GREEN -> PERIOD_GREEN
- J3: footprint Connector_PinSocket_2.54mm:PinSocket_1x04_P2.54mm_Horizontal -> Connector_PinSocket_2.54mm:PinSocket_1x04_P2.54mm_Vertical
- R1, R2, R3, R4, R5, R6, R7, R8: footprint Resistor_SMD:R_1206_3216Metric_Pad1.30x1.75mm_HandSolder -> Resistor_SMD:R_0805_2012Metric_Pad1.20x1.40mm_HandSolder
- moved R5 87.2 mm to (159.0, 132.3), turned to 90 degrees
- moved R1 76.1 mm to (152.0, 110.5), turned to -90 degrees
- moved R4 74.8 mm to (128.0, 132.5), turned to 90 degrees
- moved C6 72.5 mm to (150.0, 108.5), turned to -90 degrees
- moved C11 72.3 mm to (142.0, 132.3), turned to -90 degrees
- moved C12 71.6 mm to (145.0, 132.3), turned to -90 degrees
- moved R8 67.4 mm to (153.5, 120.0), turned to -90 degrees
- moved SW2 66.1 mm to (152.0, 132.5), turned to 180 degrees
- moved C4 64.7 mm to (154.0, 86.5)
- moved R7 63.3 mm to (139.7, 123.5), turned to 180 degrees
- moved C8 61.6 mm to (139.0, 110.8), turned to -90 degrees
- moved Y1 57.9 mm to (135.0, 108.5), turned to 90 degrees
- moved C9 55.3 mm to (130.5, 113.0), turned to 90 degrees
- moved C3 54.0 mm to (150.0, 63.5), turned to 180 degrees
- moved J1 49.5 mm to (152.0, 54.0)
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Connections:
- U2 pad 8: ENABLE_KEY -> PERIOD_KEY
- U2 pad 9: PERIOD_KEY -> ENABLE_KEY
Routing:
- net GND: track 0.00 -> 197.4 mm, vias 0 -> 14
- net +3V3: track 0.00 -> 147.4 mm, vias 0 -> 4
- net +12V: track 0.00 -> 58.9 mm, vias 0 -> 2
- net +BATT: track 0.00 -> 44.3 mm
- net ENABLE_KEY: track 0.00 -> 39.5 mm
- net PERIOD_KEY: track 0.00 -> 38.9 mm
- net INJ_PULSES: track 0.00 -> 32.2 mm
- net #RST: track 0.00 -> 25.8 mm, vias 0 -> 2
- net Net-(D2-A): track 0.00 -> 19.2 mm
- net Net-(U2-PF1): track 0.00 -> 18.6 mm
- net PERIOD_LED: track 0.00 -> 17.9 mm
- net ENABLE_LED: track 0.00 -> 13.3 mm
- net Net-(U2-PF0): track 0.00 -> 12.3 mm
- net SWDIO: track 0.00 -> 10.6 mm
- net SWCLK: track 0.00 -> 9.81 mm
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- added copper zone on B.Cu, net GND
- added copper zone on F.Cu, net GND
Other:
- board outline added: 35 x 90 mm
- board text added: "DIESEL"
- board text added: "ENABLE"
- board text added: "INJECTOR"
- board text added: "PERIOD"
- board text added: "POWER"
- board text added: "PWR"
- board text added: "TESTER"
- board text added: "trwgQ26xxx 2025"
